File: IMU.brd (EAGLE design)
At the start: 53.3 x 68.6 mm, 80 parts, among them IC1 LM358D, J2 4POS_SPDT_DIP, T1 PMOS, Y1 RESONATORSMD, Y2 16MHz

Commit message: Made some fixes for missing libraries
Parts:
- C14, C15: device rcl:C1210 -> rcl:C1206
- C4: device rcl:C0603 -> rcl:C0805
- L2: device SparkFun:0805 -> SparkFun-Passives:0805
- Y1: value RESONATORSMD -> 16MHz
- moved C14 4.45 mm to (15.5, 63.4), turned to 90 degrees
- moved C15 0.63 mm to (27.3, 57.4)
- moved C4 0.36 mm to (19.1, 37.3)
- moved R6 0.25 mm to (24.0, 24.6)
- moved Y1 0.13 mm to (26.2, 24.6)
Routing:
- net GND: track 61.2 -> 52.9 mm, vias 94 -> 96
- net USBVCC: track 26.6 -> 23.8 mm, vias 2 -> 0
- net +5V: track 267.3 -> 269.4 mm
- net VIN: track 71.4 -> 72.4 mm
- net SETC: track 3.05 -> 2.30 mm
- net SETP: track 14.0 -> 13.4 mm
- net XTAL1: track 5.98 -> 5.38 mm
- net XTAL2: track 6.38 -> 5.79 mm
