File: IMU.sch (EAGLE design)
At the start: 71 parts, among them IC1 LM358D, J2 4POS_SPDT_DIP, T1 PMOS, Y1 RESONATORSMD, Y2 16MHz

Commit message: Made some fixes for missing libraries
Parts:
- C14, C15: device rcl:C-EUC1210 -> rcl:C-EUC1206
- C21, C23, C4, C6: device rcl:C-EUC0603 -> rcl:C-EUC0805
- L2: device rcl:L-USL4532C -> SparkFun-Passives:INDUCTOR0805
- R10, R11, R12, R13, R4: device rcl:R-US_R1210W -> rcl:R-US_R0603
- Y1: value RESONATORSMD -> 16MHz
Other:
- moved on the sheet: Y1
